File: Hardware/PCB/Flight_Control/Flight_Control.kicad_sch (KiCad schematic)
At the start: 8 parts, among them U1 STM32F405RGTx, U2 BMP390, U3 ICM-42688-P

Commit message: schematic_pcb
Parts:
- added C10, C6: 4.7u, Capacitor_SMD:C_0402_1005Metric, symbol Device:C
- added C11, C12, C13, C32, C33, C34, C35, C7, C8, C9: 100n, Capacitor_SMD:C_0402_1005Metric, symbol Device:C
- added C14, C15, C29, C30: 2.2u, Capacitor_SMD:C_0402_1005Metric, symbol Device:C
- added C16: 0.01u, Capacitor_SMD:C_0402_1005Metric, symbol Device:C
- added C17, C28: 0.1u, Capacitor_SMD:C_0402_1005Metric, symbol Device:C
- added C18, C20: 47u, Capacitor_SMD:C_0402_1005Metric, symbol Device:C
- added C19: 6.8u, Capacitor_SMD:C_0402_1005Metric, symbol Device:C
- added C21: 39pF, Capacitor_SMD:C_0402_1005Metric, symbol Device:C
- added C22, C37: 10n, Capacitor_SMD:C_0402_1005Metric, symbol Device:C
- added C23: 10u, Capacitor_SMD:C_0402_1005Metric, symbol Device:C
- added C24, C25, C26, C27, C36: 1u, Capacitor_SMD:C_0402_1005Metric, symbol Device:C
- added C31: 5p, Capacitor_SMD:C_0402_1005Metric, symbol Device:C
- added D1: BZV55B5V6, Diode_SMD:D_MiniMELF, symbol Diode:BZV55B5V6
- added D2, D6: PTVS5V0Z1USK, Diode_SMD:Nexperia_DSN1608-2_1.6x0.8mm, symbol Diode:PTVS5V0Z1USK
- added D3, D4: D, Diode_SMD:D_0402_1005Metric, symbol Device:D
- added D5: PTVS10VZ1USK, Diode_SMD:Nexperia_DSN1608-2_1.6x0.8mm, symbol Diode:PTVS10VZ1USK
- added H1, H2, H3, H4: MountingHole_Pad, MountingHole:MountingHole_3.2mm_M3, symbol Mechanical:MountingHole_Pad
- added IC1, IC2: AP7365-33SNG-7, maker:AP2301SN7, symbol maker:AP7365-33SNG-7
- added J1: B4B-XH-A, maker:JST_B4B-XH-A, symbol maker:B4B-XH-A
- added J2: USB4110GFA, maker:GCT_USB4110GFA, symbol maker:USB4110GFA
- added J3: S2B-PH-K-SLFSN, maker:CONN_S2B-PH-K-S_JST, symbol maker:S2B-PH-K-SLFSN
- added L1: 8.2u, Inductor_SMD:L_0402_1005Metric, symbol Device:L
- added L2: 39n, Inductor_SMD:L_0402_1005Metric, symbol Device:L
- added R1, R2: 5.1k, Resistor_SMD:R_0402_1005Metric, symbol Device:R
- added R10: 13k, Resistor_SMD:R_0402_1005Metric, symbol Device:R
- added R11, R13, R14, R15, R16, R17: 10k, Resistor_SMD:R_0402_1005Metric, symbol Device:R
- added R12: 4.5k, Resistor_SMD:R_0402_1005Metric, symbol Device:R
- added R3, R4, R7: R, Resistor_SMD:R_0402_1005Metric, symbol Device:R
- added R5: 49.9, Resistor_SMD:R_0402_1005Metric, symbol Device:R
- added R6: 1k, Resistor_SMD:R_0402_1005Metric, symbol Device:R
- added R8: 53.6k, Resistor_SMD:R_0402_1005Metric, symbol Device:R
- added R9: 10.2k, Resistor_SMD:R_0402_1005Metric, symbol Device:R
- added SW1: 1825910-6, maker:SW4_1825910-B_TEC, symbol maker:1825910-6
- added U4: USBLC6-2SC6, Package_TO_SOT_SMD:SOT-23-6, symbol Power_Protection:USBLC6-2SC6
- added U5: TPS54361DPRR, maker:DPR0010A_TEX, symbol maker:TPS54361DPRR
- C1, C2, C3, C4, C5: footprint (none) -> Capacitor_SMD:C_0402_1005Metric
- U3: footprint LGA14_2P5X3X0P91_TDK -> maker:LGA14_2P5X3X0P91_TDK
Connections:
- net CSB: now also U1.50 (PA15)
- net CS_IMU: now also U1.20 (PA4)
- net GND: now also C1.1, U1.12 (VSSA), U1.18 (VSS), U1.63 (VSS), C10.2, C11.2, C12.2, C13.2, C14.2, C15.2, C16.2, C18.2, C19.2, C20.2, C21.2, C22.2, C23.2, C24.2, C25.2, C26.2, C27.2, C28.2, C29.2, C30.2, C31.2, C32.2, C33.2, C34.2, C35.2, C36.2, C37.2, C6.2, C7.2, C8.2, C9.2, D1.2 (A), D2.2 (A), D5.2 (A), D6.2 (A), H1.1, H2.1, H3.1, H4.1, IC1.2 (GND), IC1.7 (EP), IC2.2 (GND), IC2.7 (EP), J1.4, J2.A1/B12 (GND), J2.B1/A12 (GND), J2.S1 (GND), J2.S2 (GND), J2.S3 (GND), J2.S4 (GND), J3.2 (-), R1.1, R12.2, R14.2, R16.2, R17.2, R2.2, R4.2, R7.2, R9.2, U4.2 (GND), U5.11 (PAD), U5.8 (GND); no longer C1.2
- net INTB: now also U1.24 (PC4), R17.1
- net INT_IMU: now also U1.10 (PC2), R16.1
- net SCK: now also U1.55 (PB3)
- net SDI: now also U1.23 (PA7)
- net SDO: now also U1.56 (PB4)
- net +3.3V MCU: now reaches U1.1 (VBAT)
- net +3.3V MCU: now also U1.19 (VDD), U1.32 (VDD), U1.48 (VDD), U1.64 (VDD), C32.1, C33.1, C6.1, C7.1, C8.1, C9.1, L2.1, SW1.1
- net +3.3V MCU A: now reaches U1.13 (VDDA)
- net +3.3V MCU A: now also C36.1, C37.1, L2.2
- net ADC_BAT: now reaches U1.26 (PB0)
- net ADC_BAT: now also C31.1, R11.2, R12.1
- net at U1.31 (VCAP_1): now also C29.1
- net RX_Rad: now reaches U1.42 (PA9)
- net RX_Rad: now also J1.2
- net TX_Rad: now reaches U1.43 (PA10)
- net TX_Rad: now also J1.1
- net USB_DM: now reaches U1.44 (PA11)
- net USB_DM: now also U4.4 (I/O2)
- net USB_DP: now reaches U1.45 (PA12)
- net USB_DP: now also U4.3 (I/O2)
- net at U1.47 (VCAP_2): now also C30.1
- net BOOT: now reaches U1.60 (BOOT0)
- net BOOT: now also SW1.3
- net at U1.7 (NRST): now also C28.1
- net 3.3V B renamed +3.3V P
- net +3.3V P: now also C1.2, C10.1, C11.1, C12.1, C13.1, C27.1, C34.1, C35.1, D6.1 (K), IC2.4 (OUT); no longer C1.1
- new net: C18.1, C20.1, L1.2, R5.1, R6.1, U5.10 (PWRGD)
- new net: C19.1, R10.2
- new net: R5.2, R8.1
- new net: R8.2, R9.1, U5.6 (FB)
- new net: R3.2, R7.1, U5.3 (EN)
- new net: C17.2, D1.1 (K), L1.1, U5.9 (SW)
- new net: C21.1, R10.1, U5.7 (COMP)
- new net: C23.1, R14.1, SW1.4
- new net: IC1.1 (EN), R13.1
- new net: C16.1, U5.4 (SS_TR)
- new net: J2.B5 (CC2), R2.1
- new net: IC2.1 (EN), R15.1
- new net: J2.A5 (CC1), R1.2
- new net: R4.1, U5.5 (RT_CLK)
- new net: C17.1, U5.1 (BOOT)
- new net +3.3V A: C24.1, D2.1 (K), IC1.4 (OUT)
- new net +5V: C26.1, D4.2 (A), IC2.3 (IN), J1.3, R15.2, R6.2
- new net +5V MCU: C25.1, D3.1 (K), IC1.3 (IN), R13.2
- new net +5V MCU+IMU: D4.1 (K)
- new net +7.4V: C14.1, C15.1, C22.1, D5.1 (K), J3.1 (+), R11.1, R3.1, U5.2 (VIN)
- new net D+: J2.A6 (DP1), J2.B6 (DP2), U4.1 (I/O1)
- new net D-: J2.A7 (DN1), J2.B7 (DN2), U4.6 (I/O1)
- new net V_USB: D3.2 (A), J2.A4/B9 (VBUS), J2.B4/A9 (VBUS), U4.5 (VBUS)
- no-connect marks 0 -> 46
Other:
- note added: "Battery 2S"
- note added: "Bootload mode"
- note added: "Buck +5V"
- note added: "INTERRUPT"
- note added: "MCU - STM32F405RGT6"
- note added: "Mounting holes"
- note added: "Radio Interface 5V + UART"
- note added: "Regu(s) +3.3V"
- note added: "SPI"
- note added: "UART RADIO"
- note added: "USB Interface"
- note added: "USBC DATA"
- moved on the sheet: C1, U1

Commit message: pcb_root_unfinished
Parts:
- removed H1, H2, H3, H4: MountingHole_Pad, MountingHole:MountingHole_3.2mm_M3, symbol Mechanical:MountingHole_Pad
- added H1, H2, H3, H4: MountingHole_Pad_MP, MountingHole:MountingHole_2.2mm_M2, symbol Mechanical:MountingHole_Pad_MP
- added J4: B4B-XH-A, maker:JST_B4B-XH-A, symbol maker:B4B-XH-A
Connections:
- net +5V MCU+IMU is gone; now on net +5V MCU: D4.1 (K)
- net GND: now also H1.MP, H2.MP, H3.MP, H4.MP
- net M1: now reaches U1.14 (PA0)
- net M1: now also J4.1
- net M2: now reaches U1.15 (PA1)
- net M2: now also J4.2
- net M3: now reaches U1.16 (PA2)
- net M3: now also J4.3
- net M4: now reaches U1.17 (PA3)
- net M4: now also J4.4
- no-connect marks 46 -> 42
Other:
- note added: "ESC Command"
- moved on the sheet: C31
